Commit message: Fix FAST-LIO simulation Init Stability & Update Docs
- Reset FAST-LIO config to disable internal time sync and use raw points
- Fix robot spawn height to z=-1.5 to prevent IMU impact shock
- Remove redundant filter scripts
- Update README with Jazzy-to-Humble details and Troubleshooting log

File: setup/robot.urdf.xacro (robot description, xacro)
@@ -24,4 +24,9 @@
     <origin xyz="0.0 0.0 0.0" rpy="0.0 0.0 0.0"/>
   </xacro:intel_realsense>
+  <!-- imu_0 -->
+  <xacro:include filename="$(find clearpath_sensors_description)/urdf/microstrain_imu.urdf.xacro"/>
+  <xacro:microstrain_imu name="imu_0" parent_link="default_mount" update_rate="100">
+    <origin xyz="0.0 0.0 0.0" rpy="0.0 0.0 0.0"/>
+  </xacro:microstrain_imu>
   <!-- Manipulators -->
   <!-- Extras -->
